Commit message: Add files via upload

File: body/hexapod.urdf (robot description, URDF)
Before this commit: robot Hexapod_1, 25 links, 24 joints
Links:
- link base1: mass None -> 0.198; geometry collision mesh filename=new_parts5//base1.dae; collision mesh filename=new_parts5//base2.dae
- link joint1: mass None -> 0.015; geometry collision mesh filename=new_parts5//joint1.dae; visual mesh filename=new_parts5//joint1.dae
- link joint2: mass None -> 0.015; geometry collision mesh filename=new_parts5//joint1.dae; visual mesh filename=new_parts5//joint1.dae
- link joint3: mass None -> 0.015; geometry collision mesh filename=new_parts5//joint1.dae; visual mesh filename=new_parts5//joint1.dae
- link joint4: mass None -> 0.015; geometry collision mesh filename=new_parts5//joint1.dae; visual mesh filename=new_parts5//joint1.dae
- link joint5: mass None -> 0.015; geometry collision mesh filename=new_parts5//joint1.dae; visual mesh filename=new_parts5//joint1.dae
- link joint6: mass None -> 0.015; geometry collision mesh filename=new_parts5//joint1.dae; visual mesh filename=new_parts5//joint1.dae
- link leg1: mass None -> 0.076; geometry collision mesh filename=new_parts5//Legmotor456.dae; visual mesh filename=new_parts5//Legmotor456.dae
- link leg2: mass None -> 0.076; geometry collision mesh filename=new_parts5//Legmotor456.dae; visual mesh filename=new_parts5//Legmotor456.dae
- link leg3: mass None -> 0.076; geometry collision mesh filename=new_parts5//Legmotor456.dae; visual mesh filename=new_parts5//Legmotor456.dae
- link leg4: mass None -> 0.076; geometry collision mesh filename=new_parts5//Legmotor123.dae; visual mesh filename=new_parts5//Legmotor123.dae
- link leg5: mass None -> 0.076; geometry collision mesh filename=new_parts5//Legmotor123.dae; visual mesh filename=new_parts5//Legmotor123.dae
- link leg6: mass None -> 0.076; geometry collision mesh filename=new_parts5//Legmotor123.dae; visual mesh filename=new_parts5//Legmotor123.dae
- link motor1_1: mass None -> 0.055; geometry collision mesh filename=new_parts5//motor.dae; visual mesh filename=new_parts5//motor.dae
- link motor1_2: mass None -> 0.055; geometry collision mesh filename=new_parts5//motor1.dae; visual mesh filename=new_parts5//motor1.dae
- link motor2_1: mass None -> 0.055; geometry collision mesh filename=new_parts5//motor.dae; visual mesh filename=new_parts5//motor.dae
- link motor2_2: mass None -> 0.055; geometry collision mesh filename=new_parts5//motor1.dae; visual mesh filename=new_parts5//motor1.dae
- link motor3_1: mass None -> 0.055; geometry collision mesh filename=new_parts5//motor.dae; visual mesh filename=new_parts5//motor.dae
- link motor3_2: mass None -> 0.055; geometry collision mesh filename=new_parts5//motor1.dae; visual mesh filename=new_parts5//motor1.dae
- link motor4_1: mass None -> 0.055; geometry collision mesh filename=new_parts5//motor.dae; visual mesh filename=new_parts5//motor.dae
- link motor4_2: mass None -> 0.055; geometry collision mesh filename=new_parts5//motor1.dae; visual mesh filename=new_parts5//motor1.dae
- link motor5_1: mass None -> 0.055; geometry collision mesh filename=new_parts5//motor.dae; visual mesh filename=new_parts5//motor.dae
- link motor5_2: mass None -> 0.055; geometry collision mesh filename=new_parts5//motor1.dae; visual mesh filename=new_parts5//motor1.dae
- link motor6_1: mass None -> 0.055; geometry collision mesh filename=new_parts5//motor.dae; visual mesh filename=new_parts5//motor.dae
- link motor6_2: mass None -> 0.055; geometry collision mesh filename=new_parts5//motor1.dae; visual mesh filename=new_parts5//motor1.dae
